Commit message: changed ur_gripper_moveit_config to ur_robotiq_moveit_config

File: ur_robotiq_description/urdf/ur5e_with_robotiq_hande.urdf (robot description, URDF)
Before this commit: robot ur5e_with_robotiq_hande, 16 links, 15 joints
Links:
- removed link world
Joints:
- removed joint world_joint
- joint hande_left_finger_joint: limit lower=0 upper=0.025 effort=130 velocity=0.15 -> (none); type prismatic -> fixed
- joint hande_right_finger_joint: limit lower=0 upper=0.025 effort=130 velocity=0.15 -> (none); mimic joint=hande_left_finger_joint multiplier=1 offset=0 -> (none); type prismatic -> fixed

File: ur_robotiq_moveit_config/config/ur5e_with_robotiq_hande.ros2_control.xacro (robot description, xacro)
@@ -50,11 +50,4 @@
                 <state_interface name="velocity"/>
             </joint>
-            <joint name="hande_left_finger_joint">
-                <command_interface name="position"/>
-                <state_interface name="position">
-                  <param name="initial_value">${initial_positions['hande_left_finger_joint']}</param>
-                </state_interface>
-                <state_interface name="velocity"/>
-            </joint>
         </ros2_control>
     </xacro:macro>
